File: small.sch (EAGLE design)
At the start: 4 parts, among them U1 SN74LS241N

Commit message: Add files via upload
Parts:
- removed JP1: (no value), adafruit:PINHD-1X6
- added J2: 53375-0610, wire to board_molex:53375-0610
- J1: value (none) -> 53253-0370; device Wurth_Connectors_WR-WTB:62000311622 -> xl320_molex:53253-0370
Connections:
- net 5V: now also J2.2; no longer JP1.2
- net 7.4V: now also J2.1; no longer JP1.1
- net DATA_CONTROL: now also J2.4; no longer JP1.4
- net GND: now also J2.3; no longer JP1.3
- net RX: now also J2.6; no longer JP1.6
- net TX: now also J2.5; no longer JP1.5
Changed lines of the file:
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@@
 <parts>
 <part name="U1" library="74LS241" deviceset="SN74LS241N" device=""/>
-<part name="J1" library="Wurth_Connectors_WR-WTB" library_urn="urn:adsk.eagle:library:15818693" deviceset="62000311622" device="" package3d_urn="urn:adsk.eagle:package:15819073/2"/>
-<part name="JP1" library="adafruit" deviceset="PINHD-1X6" device=""/>
 <part name="R1" library="adafruit" deviceset="R-US_" device="M0805" value="10k"/>
+<part name="J2" library="wire to board_molex" deviceset="53375-0610" device=""/>
+<part name="J1" library="xl320_molex" deviceset="53253-0370" device=""/>
 </parts>
 <sheets>
@@
 <instances>
 <instance part="U1" gate="A" x="25.4" y="58.42"/>
-<instance part="J1" gate="G$1" x="48.26" y="20.32"/>
-<instance part="JP1" gate="A" x="114.3" y="17.78"/>
 <instance part="R1" gate="G$1" x="15.24" y="53.34"/>
+<instance part="J2" gate="G$1" x="129.54" y="20.32" rot="R270"/>
+<instance part="J1" gate="G$1" x="45.72" y="12.7" smashed="yes" rot="R90">
+<attribute name="NAME" x="48.26" y="24.13" size="1.778" layer="95" rot="R90" align="center-left"/>
+</instance>
 </instances>
 <busses>
@@
 <wire x1="111.76" y1="22.86" x2="104.14" y2="22.86" width="0.1524" layer="91"/>
 <label x="104.14" y="22.86" size="1.778" layer="95" rot="R180" xref="yes"/>
-<pinref part="JP1" gate="A" pin="2"/>
+<pinref part="J2" gate="G$1" pin="2"/>
+<wire x1="111.76" y1="22.86" x2="127" y2="22.86" width="0.1524" layer="91"/>
+<wire x1="127" y1="22.86" x2="127" y2="20.32" width="0.1524" layer="91"/>
 </segment>
 <segment>
@@
 </segment>
 <segment>
-<pinref part="J1" gate="G$1" pin="1"/>
-<wire x1="50.8" y1="15.24" x2="50.8" y2="12.7" width="0.1524" layer="91"/>
-<label x="50.8" y="12.7" size="1.778" layer="95" rot="R270" xref="yes"/>
+<wire x1="124.46" y1="20.32" x2="104.14" y2="20.32" width="0.1524" layer="91"/>
+<label x="104.14" y="20.32" size="1.778" layer="95" rot="R180" xref="yes"/>
+<pinref part="J2" gate="G$1" pin="3"/>
 </segment>
 <segment>
-<wire x1="111.76" y1="20.32" x2="104.14" y2="20.32" width="0.1524" layer="91"/>
-<label x="104.14" y="20.32" size="1.778" layer="95" rot="R180" xref="yes"/>
-<pinref part="JP1" gate="A" pin="3"/>
+<pinref part="J1" gate="G$1" pin="1"/>
+<wire x1="45.72" y1="12.7" x2="45.72" y2="10.16" width="0.1524" layer="91"/>
+<label x="45.72" y="10.16" size="1.778" layer="95" rot="R270" xref="yes"/>
 </segment>
 </net>
@@
 <wire x1="111.76" y1="17.78" x2="104.14" y2="17.78" width="0.1524" layer="91"/>
 <label x="104.14" y="17.78" size="1.778" layer="95" rot="R180" xref="yes"/>
-<pinref part="JP1" gate="A" pin="4"/>
+<wire x1="111.76" y1="17.78" x2="119.38" y2="17.78" width="0.1524" layer="91"/>
+<wire x1="119.38" y1="17.78" x2="119.38" y2="0" width="0.1524" layer="91"/>
+<wire x1="119.38" y1="0" x2="119.38" y2="-7.62" width="0.1524" layer="91"/>
+<wire x1="119.38" y1="-7.62" x2="129.54" y2="-7.62" width="0.1524" layer="91"/>
+<pinref part="J2" gate="G$1" pin="4"/>
+<wire x1="129.54" y1="-7.62" x2="129.54" y2="0" width="0.1524" layer="91"/>
 </segment>
 </net>
@@
 <segment>
 <pinref part="J1" gate="G$1" pin="3"/>
-<wire x1="45.72" y1="15.24" x2="45.72" y2="12.7" width="0.1524" layer="91"/>
-<label x="45.72" y="12.7" size="1.778" layer="95" rot="R270" xref="yes"/>
+<wire x1="50.8" y1="12.7" x2="53.34" y2="12.7" width="0.1524" layer="91"/>
+<label x="53.34" y="12.7" size="1.778" layer="95" xref="yes"/>
 </segment>
 </net>
@@
 <wire x1="111.76" y1="12.7" x2="104.14" y2="12.7" width="0.1524" layer="91"/>
 <label x="104.14" y="12.7" size="1.778" layer="95" rot="R180" xref="yes"/>
-<pinref part="JP1" gate="A" pin="6"/>
+<wire x1="111.76" y1="12.7" x2="111.76" y2="-2.54" width="0.1524" layer="91"/>
+<wire x1="111.76" y1="-2.54" x2="124.46" y2="-2.54" width="0.1524" layer="91"/>
+<pinref part="J2" gate="G$1" pin="6"/>
+<wire x1="124.46" y1="-2.54" x2="124.46" y2="0" width="0.1524" layer="91"/>
 </segment>
 </net>
@@
 <wire x1="111.76" y1="15.24" x2="104.14" y2="15.24" width="0.1524" layer="91"/>
 <label x="104.14" y="15.24" size="1.778" layer="95" rot="R180" xref="yes"/>
-<pinref part="JP1" gate="A" pin="5"/>
+<wire x1="111.76" y1="15.24" x2="116.84" y2="15.24" width="0.1524" layer="91"/>
+<wire x1="116.84" y1="15.24" x2="116.84" y2="12.7" width="0.1524" layer="91"/>
+<wire x1="116.84" y1="12.7" x2="116.84" y2="-5.08" width="0.1524" layer="91"/>
+<wire x1="116.84" y1="-5.08" x2="119.38" y2="-5.08" width="0.1524" layer="91"/>
+<wire x1="119.38" y1="-5.08" x2="127" y2="-5.08" width="0.1524" layer="91"/>
+<pinref part="J2" gate="G$1" pin="5"/>
+<wire x1="127" y1="-5.08" x2="127" y2="0" width="0.1524" layer="91"/>
 </segment>
 </net>
 <net name="7.4V" class="0">
 <segment>
-<pinref part="J1" gate="G$1" pin="2"/>
-<wire x1="48.26" y1="15.24" x2="48.26" y2="12.7" width="0.1524" layer="91"/>
-<label x="48.26" y="12.7" size="1.778" layer="95" rot="R270" xref="yes"/>
+<wire x1="111.76" y1="25.4" x2="104.14" y2="25.4" width="0.1524" layer="91"/>
+<label x="104.14" y="25.4" size="1.778" layer="95" rot="R180" xref="yes"/>
+<pinref part="J2" gate="G$1" pin="1"/>
+<wire x1="111.76" y1="25.4" x2="129.54" y2="25.4" width="0.1524" layer="91"/>
+<wire x1="129.54" y1="25.4" x2="129.54" y2="20.32" width="0.1524" layer="91"/>
 </segment>
 <segment>
-<wire x1="111.76" y1="25.4" x2="104.14" y2="25.4" width="0.1524" layer="91"/>
-<label x="104.14" y="25.4" size="1.778" layer="95" rot="R180" xref="yes"/>
-<pinref part="JP1" gate="A" pin="1"/>
+<pinref part="J1" gate="G$1" pin="2"/>
+<wire x1="48.26" y1="12.7" x2="48.26" y2="7.62" width="0.1524" layer="91"/>
+<label x="48.26" y="7.62" size="1.778" layer="95" xref="yes"/>
 </segment>
 </net>
@@
 </schematic>
 </drawing>
-<compatibility>
-<note version="8.2" severity="warning">
-Since Version 8.2, EAGLE supports online libraries. The ids
-of those online libraries will not be understood (or retained)
-with this version.
-</note>
-<note version="8.3" severity="warning">
-Since Version 8.3, EAGLE supports URNs for individual library
-assets (packages, symbols, and devices). The URNs of those assets
-will not be understood (or retained) with this version.
-</note>
-<note version="8.3" severity="warning">
-Since Version 8.3, EAGLE supports the association of 3D packages
-with devices in libraries, schematics, and board files. Those 3D
-packages will not be understood (or retained) with this version.
-</note>
-</compatibility>
 </eagle>
