File: small.sch (EAGLE design)
At the start: 4 parts, among them U1 SN74LS241N

Commit message: Add files via upload
Parts:
- removed JP1: (no value), adafruit:PINHD-1X6
- added C8: 10uF, adafruit:C-USC0805
- added C9: 1uF, Common-Parts-Library-Eagle:CC0603KRX7R9BB104
- added J2: 53375-0610, wire to board_molex:53375-0610
- added J3, J4, J5, J6: F-1X07-SIP-100-32, con-headers-jp:F-1X07-SIP-100-32
- added J7: CLM-107-02-L-D-A, CLM-107-02-L-D-A:CLM-107-02-L-D-A
- added J8: F-2X07-DIL-100, con-headers-jp:F-2X07-DIL-100
- added U$1: IMU, IMU:IMU
- J1: value (none) -> 53253-0370; device Wurth_Connectors_WR-WTB:62000311622 -> xl320_molex:53253-0370; OC_FARNELL (none) -> unknown
- R1: MF (none) -> VISHAY; MPN (none) -> CRCW080510K0JNEA; OC_FARNELL (none) -> 1469857
- U1: MF (none) -> TEXAS INSTRUMENTS; MPN (none) -> SN74LS241N; OC_FARNELL (none) -> 3006181
Connections:
- new net 3.3V: C8.1, C9.1, J7.11, J8.10, J8.11, J8.12
- new net N$1: J4.7, U$1.PIN_4
- new net N$10: J3.5, U$1.PIN_23
- new net N$11: J3.4, U$1.PIN_22
- new net N$12: J3.3, U$1.PIN_21
- new net N$13: J3.2, U$1.PIN_20
- new net N$14: J3.1, U$1.PIN_19
- new net N$15: J6.7, U$1.PIN_18
- new net N$16: J6.6, U$1.PIN_17
- new net N$17: J6.5, U$1.PIN_16
- new net N$18: J6.4, U$1.PIN_15
- new net N$19: J6.3, U$1.PIN_14
- new net N$2: J4.6, U$1.PIN_3
- new net N$20: J6.2, U$1.PIN_13
- new net N$21: J6.1, U$1.PIN_12
- new net N$22: J5.7, U$1.PIN_11
- new net N$23: J5.6, U$1.PIN_10
- new net N$24: J5.5, U$1.PIN_9
- new net N$25: J5.4, U$1.PIN_8
- new net N$26: J5.3, U$1.PIN_7
- new net N$27: J5.2, U$1.PIN_6
- new net N$28: J5.1, U$1.PIN_5
- new net N$3: J4.5, U$1.PIN_2
- new net N$4: J4.4, U$1.PIN_1
- new net N$5: J4.3, U$1.PIN_28
- new net N$59: J7.1, J8.13
- new net N$6: J4.2, U$1.PIN_27
- new net N$60: J7.2, J8.14
- new net N$61: J7.3, J8.2
- new net N$62: J7.4, J8.4
- new net N$63: J7.5, J8.6
- new net N$64: J7.8, J8.1
- new net N$65: J7.6, J8.3
- new net N$7: J4.1, U$1.PIN_26
- new net N$8: J3.7, U$1.PIN_25
- new net N$9: J3.6, U$1.PIN_24
- net 5V: now also J2.2; no longer JP1.2
- net 7.4V: now also J2.1; no longer JP1.1
- net DATA_CONTROL: now also J2.4; no longer JP1.4
- net GND: now also C8.2, C9.2, J2.3, J7.13, J8.7, J8.8, J8.9; no longer JP1.3
- net RX: now also J2.6; no longer JP1.6
- net TX: now also J2.5; no longer JP1.5
